File: hw/JAC.kicad_sch (KiCad schematic)
At the start: 23 parts, among them J1 USB_C_Receptacle_USB2.0, Q1 AO3401A, SW1 BT0, U1 EPDM, U2 4056M, U3 RX-8025T, U4 ESP32-C3-WROOM-02

Commit message: Prepareing JAC
Parts:
- added C4: 10uF, Capacitor_SMD:C_0805_2012Metric, symbol Device:C
- J1: footprint Joke:TYPE-C-VERT -> JAC:TYPE-C-VERT
Connections:
- net +3V3: now also C4.1
- net EPD_PC: now also R2.2, U4.7 (IO8); no longer U4.3 (IO4)
- net EPD_RST: now also U4.3 (IO4); no longer R2.2, U4.7 (IO8)
- net GND: now also C4.2
Changed lines of the file:
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@@
     (stroke (width 0) (type default) (color 0 0 0 0))
   )
-  (text "墨水屏电源控制" (at 114.3 52.832 180)
+  (text "墨水屏电源控制" (at 114.046 62.992 180)
     (effects (font (size 1.27 1.27)) (justify right bottom))
   )
@@
     (effects (font (size 1.27 1.27)) (justify left bottom))
   )
-  (text "EPD RST" (at 114.046 62.992 180)
+  (text "EPD RST" (at 114.554 52.578 180)
     (effects (font (size 1.27 1.27)) (justify right bottom))
   )
@@
     (effects (font (size 1.27 1.27)) (justify right bottom))
   )
-  (label "EPD_RST" (at 116.078 61.976 0)
+  (label "EPD_RST" (at 116.078 51.816 0)
     (effects (font (size 1.27 1.27)) (justify left bottom))
   )
@@
     (effects (font (size 1.27 1.27)) (justify right bottom))
   )
-  (label "EPD_PC" (at 116.078 51.816 0)
+  (label "EPD_PC" (at 116.078 61.976 0)
     (effects (font (size 1.27 1.27)) (justify left bottom))
   )
@@
   )
   (symbol (lib_id "Device:R") (at 82.042 104.394 0) (unit 1)
-    (in_bom yes) (on_board yes) (fields_autoplaced)
+    (in_bom yes) (on_board no) (fields_autoplaced)
     (property "Reference" "R9" (id 0) (at 84.328 103.1239 0)
       (effects (font (size 1.27 1.27)) (justify left))
@@
     (pin "1")
     (pin "2")
+  )
+  (symbol (lib_id "power:GND") (at 88.138 60.198 0) (unit 1)
+    (in_bom yes) (on_board yes) (fields_autoplaced)
+    (property "Reference" "#PWR032" (id 0) (at 88.138 66.548 0)
+      (effects (font (size 1.27 1.27)) hide)
+    )
+    (property "Value" "GND" (id 1) (at 91.186 61.4679 0)
+      (effects (font (size 1.27 1.27)) (justify left))
+    )
+    (property "Footprint" "" (id 2) (at 88.138 60.198 0)
+      (effects (font (size 1.27 1.27)) hide)
+    )
+    (property "Datasheet" "" (id 3) (at 88.138 60.198 0)
+      (effects (font (size 1.27 1.27)) hide)
+    )
+    (pin "1")
   )
   (symbol (lib_id "Jumper:Jumper_2_Open") (at 202.184 107.696 0) (unit 1)
@@
     (pin "1")
   )
+  (symbol (lib_id "power:+3V3") (at 88.138 52.578 0) (unit 1)
+    (in_bom yes) (on_board yes) (fields_autoplaced)
+    (property "Reference" "#PWR031" (id 0) (at 88.138 56.388 0)
+      (effects (font (size 1.27 1.27)) hide)
+    )
+    (property "Value" "+3V3" (id 1) (at 90.17 51.3079 0)
+      (effects (font (size 1.27 1.27)) (justify left))
+    )
+    (property "Footprint" "" (id 2) (at 88.138 52.578 0)
+      (effects (font (size 1.27 1.27)) hide)
+    )
+    (property "Datasheet" "" (id 3) (at 88.138 52.578 0)
+      (effects (font (size 1.27 1.27)) hide)
+    )
+    (pin "1")
+  )
   (symbol (lib_id "power:GND") (at 111.506 111.252 270) (unit 1)
     (in_bom yes) (on_board yes) (fields_autoplaced)
@@
     (property "Reference" "J1" (id 0) (at 181.864 82.55 0))
     (property "Value" "USB_C_Receptacle_USB2.0" (id 1) (at 181.864 85.09 0))
-    (property "Footprint" "Joke:TYPE-C-VERT" (id 2) (at 185.674 105.156 0)
+    (property "Footprint" "JAC:TYPE-C-VERT" (id 2) (at 185.674 105.156 0)
       (effects (font (size 1.27 1.27)) hide)
     )
@@
     (pin "1")
   )
+  (symbol (lib_id "Device:C") (at 88.138 56.388 0) (unit 1)
+    (in_bom yes) (on_board yes) (fields_autoplaced)
+    (property "Reference" "C4" (id 0) (at 91.44 55.1179 0)
+      (effects (font (size 1.27 1.27)) (justify left))
+    )
+    (property "Value" "10uF" (id 1) (at 91.44 57.6579 0)
+      (effects (font (size 1.27 1.27)) (justify left))
+    )
+    (property "Footprint" "Capacitor_SMD:C_0805_2012Metric" (id 2) (at 89.1032 60.198 0)
+      (effects (font (size 1.27 1.27)) hide)
+    )
+    (property "Datasheet" "~" (id 3) (at 88.138 56.388 0)
+      (effects (font (size 1.27 1.27)) hide)
+    )
+    (pin "1")
+    (pin "2")
+  )
   (symbol (lib_id "JAC:ESP32-C3-WROOM-02") (at 146.812 41.656 0) (unit 1)
     (in_bom yes) (on_board yes) (fields_autoplaced)
@@
       (reference "#PWR030") (unit 1) (value "+3V3") (footprint "")
     )
+    (path "/39862cc0-1efd-48a7-b7b9-9efa626f64a2"
+      (reference "#PWR031") (unit 1) (value "+3V3") (footprint "")
+    )
+    (path "/2d83efa7-db60-46d0-a115-a6601101e23c"
+      (reference "#PWR032") (unit 1) (value "GND") (footprint "")
+    )
     (path "/3806d12d-5382-40d6-89ef-9bb14938335d"
       (reference "C1") (unit 1) (value "0.1u") (footprint "Capacitor_SMD:C_0603_1608Metric")
@@
       (reference "C3") (unit 1) (value "0.1uF") (footprint "Capacitor_SMD:C_0603_1608Metric")
     )
+    (path "/da325869-f0ef-4007-b234-69e361aac919"
+      (reference "C4") (unit 1) (value "10uF") (footprint "Capacitor_SMD:C_0805_2012Metric")
+    )
     (path "/78bc9602-2d92-4001-a79a-ec3762594f25"
-      (reference "J1") (unit 1) (value "USB_C_Receptacle_USB2.0") (footprint "Joke:TYPE-C-VERT")
+      (reference "J1") (unit 1) (value "USB_C_Receptacle_USB2.0") (footprint "JAC:TYPE-C-VERT")
     )
     (path "/7cd8afda-71f3-4c56-9528-d706c5cec949"

Commit message: hw: 4.2 inch screen variant
Parts:
- J1: footprint JAC:TYPE-C-VERT -> Connector_USB:USB_C_Receptacle_Palconn_UTC16-G
Connections:
- no-connect marks 10 -> 12
Changed lines of the file:
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@@
   (no_connect (at 111.506 101.092))
   (no_connect (at 129.286 108.712))
+  (no_connect (at 197.104 117.856))
+  (no_connect (at 197.104 120.396))
   (no_connect (at 111.506 106.172))
   (no_connect (at 129.286 111.252))
@@
     (property "Reference" "J1" (id 0) (at 181.864 82.55 0))
     (property "Value" "USB_C_Receptacle_USB2.0" (id 1) (at 181.864 85.09 0))
-    (property "Footprint" "JAC:TYPE-C-VERT" (id 2) (at 185.674 105.156 0)
+    (property "Footprint" "Connector_USB:USB_C_Receptacle_Palconn_UTC16-G" (id 2) (at 185.674 105.156 0)
       (effects (font (size 1.27 1.27)) hide)
     )
@@
     (pin "A6")
     (pin "A7")
+    (pin "A8")
     (pin "A9")
     (pin "B1")
@@
     (pin "B6")
     (pin "B7")
+    (pin "B8")
     (pin "B9")
     (pin "S1")
@@
     )
     (path "/78bc9602-2d92-4001-a79a-ec3762594f25"
-      (reference "J1") (unit 1) (value "USB_C_Receptacle_USB2.0") (footprint "JAC:TYPE-C-VERT")
+      (reference "J1") (unit 1) (value "USB_C_Receptacle_USB2.0") (footprint "Connector_USB:USB_C_Receptacle_Palconn_UTC16-G")
     )
     (path "/7cd8afda-71f3-4c56-9528-d706c5cec949"
